File: std_board.kicad_pcb (KiCad board)
At the start: 2 copper layers, 99.1 x 99.1 mm, 191 parts, among them IC1 ESP32, IC2 ACS712, IC3 L78L05, IC4 AMS1117-V, J1 Jumper, J10 J_DHT11, J11 Jumper, J12 Jumper, J13 J_PRess, J14 Jumper, J15 Jumper, J16 J_PRess, J17 Jumper, J18 Jumper, J19 Jumper, J2 Jumper, J22 Jumper, J24 Jumper, J25 Jumper, J26 Jumper, J27 Jumper, J29 Jumper, J3 Jumper, J31 Jumper, J32 Jumper, J33 Jumper, J34 Jumper, J35 Jumper, J36 Jumper, J37 Jumper, J38 Jumper, J39 Jumper, J4 Jumper, J40 Jumper, J41 Jumper, J42 Jumper, J43 Jumper, J44 Jumper, J45 Jumper, J5 Jumper, J6 J_PRess, J7 Jumper, J8 Jumper, J9 Jumper, T1 TRIAC_Micro, T2 TRIAC_Micro, T3 TRIAC_Micro, T4 NPN, T5 NPN, T6 NPN, T7 NPN, T8 PNP, T9 NPN, U1 LNK306

Commit message: gerber updated on 20210310-2044
Routing:
- net GND: track 564.0 -> 568.2 mm
Other:
- rule pad_to_mask_clearance: 0.051 -> 0
- rule solder_mask_min_width: 0.25 -> 0.4
- board text added: "std_board-0.1.0 20210310"
- board text removed: "Alfred v-1.0 202101"
