File: _autosave-std_board.kicad_pcb (KiCad board)
At the start: 2 copper layers, 99.1 x 99.1 mm, 191 parts, among them IC1 ESP32, IC2 ACS712, IC3 L78L05, IC4 AMS1117-V, J1 Jumper, J10 J_DHT11, J11 Jumper, J12 Jumper, J13 J_PRess, J14 Jumper, J15 Jumper, J16 J_PRess, J17 Jumper, J18 Jumper, J19 Jumper, J2 Jumper, J22 Jumper, J24 Jumper, J25 Jumper, J26 Jumper, J27 Jumper, J29 Jumper, J3 Jumper, J31 Jumper, J32 Jumper, J33 Jumper, J34 Jumper, J35 Jumper, J36 Jumper, J37 Jumper, J38 Jumper, J39 Jumper, J4 Jumper, J40 Jumper, J41 Jumper, J42 Jumper, J43 Jumper, J44 Jumper, J45 Jumper, J5 Jumper, J6 J_PRess, J7 Jumper, J8 Jumper, J9 Jumper, T1 TRIAC_Micro, T2 TRIAC_Micro, T3 TRIAC_Micro, T4 NPN, T5 NPN, T6 NPN, T7 NPN, T8 PNP, T9 NPN, U1 LNK306

Commit message: updates on circuit board and readme file
Routing:
- net /+3.3V: track 307.6 -> 242.8 mm
- net /K2_in: track 14.5 -> 67.9 mm
- net GND: track 565.3 -> 573.5 mm
- net P33: track 77.5 -> 71.6 mm, vias 1 -> 0
- net /DAC_1: track 122.5 -> 125.1 mm
Other:
- board text added: "- Dev_1: JTAG connector; - Dev_2: ACS712 current sensor; - Dev_3: Pressure sensor 1; - Dev_4: Pressure sensor 2; - Dev_5: DS3231 RTC; - Dev_6: DS18B20, 1 wire temp. sensor; - Dev_7: BMP150, pressure sensor; - Dev_8: DHT11 humidity sensor."
- board text added: "Current Transformer"
- board text added: "Dev_1"
- board text added: "Dev_2"
- board text added: "Dev_3"
- board text added: "Dev_4"
- board text added: "Dev_5"
- board text added: "Dev_6"
- board text added: "Dev_7"
- board text added: "Dev_8"
- board text added: "Devices pinhead onboard"
- board text added: "Invasive"
- board text added: "i_in_1"
- board text added: "i_in_2"
- board text removed: "CT: Current Transformer"
- board text removed: "JTAG"
